Commit message: First try in gazebo

File: urdf/robot_assembly(gazebo).xacro (robot description, xacro)
@@ -1,4 +1,5 @@
-<?xml version="1.0" encoding="utf-8" ?>
-<!-- This URDF was automatically created by SolidWorks to URDF Exporter! Originally created by Stephen Brawner (brawner@gmail.com)
+<?xml version="1.0" encoding="utf-8"?>
+<!-- This URDF was automatically created by SolidWorks to URDF Exporter! Originally created by
+Stephen Brawner (brawner@gmail.com)
      Commit Version: 1.6.0-4-g7f85cfe  Build Version: 1.6.7995.38578
      For more information, please see http://wiki.ros.org/sw_urdf_exporter -->
@@ -9,4 +10,15 @@
     <xacro:property name="axle_offset" value="0.05" />
     <xacro:property name="damp" value="0.7" />
+    <!-- Materials -->
+    <material name="white">
+        <color rgba="1 1 1 1" />
+    </material>
+    <material name="orange">
+        <color rgba="0.90 0.35 0.117 1" />
+    </material>
+    <material name="black">
+        <color rgba="0 0 0 1" />
+    </material>
+    <!-- WORLD-->
     <link name="world">
     </link>
@@ -15,9 +27,12 @@
         <child link="base_link" />
     </joint>
+    <!-- BASE LINK -->
     <link name="base_link">
         <inertial>
             <origin xyz="7.16570679801176E-10 0.00116092156507622 2.8893545031334E-06" rpy="0 0 0" />
             <mass value="0.0324100192967721" />
-            <inertia ixx="2.68587605210783E-05" ixy="-4.84597989563569E-14" ixz="-3.40425204588481E-13" iyy="5.34932089470888E-05" iyz="-5.34738719597888E-10" izz="2.68551853927962E-05" />
+            <inertia ixx="2.68587605210783E-05" ixy="-4.84597989563569E-14"
+                ixz="-3.40425204588481E-13" iyy="5.34932089470888E-05" iyz="-5.34738719597888E-10"
+                izz="2.68551853927962E-05" />
         </inertial>
         <visual>
@@ -26,7 +41,5 @@
                 <mesh filename="file://$(find robo_arm)/meshes/base_link.STL" />
             </geometry>
-            <material name="orange">
-                <color rgba="0.90 0.35 0.117 1" />
-            </material>
+            <material name="orange" />
         </visual>
         <collision>
@@ -37,26 +50,8 @@
         </collision>
     </link>
-    <link name="Link_1">
-<inertial>
-            <origin xyz="-0.0076360494909025 0.00173746113523518 0.0423898735296237" rpy="0 0 0" />
-            <mass value="0.190717117623996" />
-            <inertia ixx="0.00015099352493845" ixy="-1.84583823946254E-09" ixz="-4.84370294611225E-08" iyy="0.000124524225271564" iyz="2.72900596568772E-06" izz="0.00016196923748443" />
-        </inertial>
-        <visual>
-            <origin xyz="0 0 0" rpy="0 0 0" />
-            <geometry>
-                <mesh filename="file://$(find robo_arm)/meshes/Link_1.STL" />
-            </geometry>
-            <material name="">
-                <color rgba="0.90 0.35 0.117 1" />
-            </material>
-        </visual>
-        <collision>
-            <origin xyz="0 0 0" rpy="0 0 0" />
-            <geometry>
-                <mesh filename="file://$(find robo_arm)/meshes/Link_1.STL" />
-            </geometry>
-        </collision>
-    </link>
+    <gazebo reference="base_link">
+        <material>Gazebo/Orange</material>
+    </gazebo>
+    <!-- JOINT 1 -->
     <joint name="Joint_1" type="revolute">
         <origin xyz="0 0 0" rpy="0 0 -3.1319" />
@@ -66,26 +61,30 @@
         <limit lower="-1.57" upper="1.57" effort="10" velocity="50" />
     </joint>
-    <link name="Link_2">
-<inertial>
-            <origin xyz="1.5639E-05 0.00028327 -0.082259" rpy="0 0 0" />
-            <mass value="0.084639" />
-            <inertia ixx="0.00014025" ixy="-4.6225E-12" ixz="-3.076E-07" iyy="0.00012793" iyz="1.6402E-07" izz="3.0857E-05" />
-        </inertial>
-        <visual>
-            <origin xyz="0 0 0" rpy="0 0 0" />
-            <geometry>
-                <mesh filename="file://$(find robo_arm)/meshes/Link_2.STL" />
-            </geometry>
-            <material name="">
-                <color rgba="0.90 0.35 0.117 1" />
-            </material>
-        </visual>
-        <collision>
-            <origin xyz="0 0 0" rpy="0 0 0" />
-            <geometry>
-                <mesh filename="file://$(find robo_arm)/meshes/Link_2.STL" />
-            </geometry>
-        </collision>
-    </link>
+    <link name="Link_1">
+        <inertial>
+            <origin xyz="-0.0076360494909025 0.00173746113523518 0.0423898735296237" rpy="0 0 0" />
+            <mass value="0.190717117623996" />
+            <inertia ixx="0.00015099352493845" ixy="-1.84583823946254E-09"
+                ixz="-4.84370294611225E-08" iyy="0.000124524225271564" iyz="2.72900596568772E-06"
+                izz="0.00016196923748443" />
+        </inertial>
+        <visual>
+            <origin xyz="0 0 0" rpy="0 0 0" />
+            <geometry>
+                <mesh filename="file://$(find robo_arm)/meshes/Link_1.STL" />
+            </geometry>
+            <material name="orange" />
+        </visual>
+        <collision>
+            <origin xyz="0 0 0" rpy="0 0 0" />
+            <geometry>
+                <mesh filename="file://$(find robo_arm)/meshes/Link_1.STL" />
+            </geometry>
+        </collision>
+    </link>
+    <gazebo reference="Link_1">
+        <material>Gazebo/Orange</material>
+    </gazebo>
+    <!-- JOINT 2 -->
     <joint name="Joint_2" type="revolute">
         <origin xyz="0 0 0.071305" rpy="3.1416 -0.64542 1.5708" />
@@ -95,26 +94,29 @@
         <limit lower="-1.65" upper="0.35" effort="10" velocity="50" />
     </joint>
-    <link name="Link_3">
-<inertial>
-            <origin xyz="1.56358976851345E-05 -0.000283205718507318 -0.0822589976475606" rpy="0 0 0" />
-            <mass value="0.0846391903579548" />
-            <inertia ixx="0.000140247302733448" ixy="-4.69358368842248E-12" ixz="-3.07601656051575E-07" iyy="0.000127934879343709" iyz="-1.64072771614451E-07" izz="3.08569655735298E-05" />
-        </inertial>
-        <visual>
-            <origin xyz="0 0 0" rpy="0 0 0" />
-            <geometry>
-                <mesh filename="file://$(find robo_arm)/meshes/Link_3.STL" />
-            </geometry>
-            <material name="">
-                <color rgba="0.90 0.35 0.117 1" />
-            </material>
-        </visual>
-        <collision>
-            <origin xyz="0 0 0" rpy="0 0 0" />
-            <geometry>
-                <mesh filename="file://$(find robo_arm)/meshes/Link_3.STL" />
-            </geometry>
-        </collision>
-    </link>
+    <link name="Link_2">
+        <inertial>
+            <origin xyz="1.5639E-05 0.00028327 -0.082259" rpy="0 0 0" />
+            <mass value="0.084639" />
+            <inertia ixx="0.00014025" ixy="-4.6225E-12" ixz="-3.076E-07" iyy="0.00012793"
+                iyz="1.6402E-07" izz="3.0857E-05" />
+        </inertial>
+        <visual>
+            <origin xyz="0 0 0" rpy="0 0 0" />
+            <geometry>
+                <mesh filename="file://$(find robo_arm)/meshes/Link_2.STL" />
+            </geometry>
+            <material name="orange" />
+        </visual>
+        <collision>
+            <origin xyz="0 0 0" rpy="0 0 0" />
+            <geometry>
+                <mesh filename="file://$(find robo_arm)/meshes/Link_2.STL" />
+            </geometry>
+        </collision>
+    </link>
+    <gazebo reference="Link_2">
+        <material>Gazebo/Orange</material>
+    </gazebo>
+    <!-- JOINT 3 -->
     <joint name="Joint_3" type="revolute">
         <origin xyz="0 0 -0.12503" rpy="0 1.5181 -3.1416" />
@@ -124,26 +126,30 @@
         <limit lower="-3.14" upper="0.14" effort="10" velocity="50" />
     </joint>
-    <link name="Link_4">
-<inertial>
-            <origin xyz="-0.000290289833333423 0.0355291858374829 0.00215430200212582" rpy="0 0 0" />
-            <mass value="0.0395556566949035" />
-            <inertia ixx="2.27747448686024E-05" ixy="-1.15013948411467E-07" ixz="-7.6137139609455E-10" iyy="1.92306725633858E-05" iyz="-3.31159527434926E-07" izz="3.22545102910992E-05" />
-        </inertial>
-        <visual>
-            <origin xyz="0 0 0" rpy="0 0 0" />
-            <geometry>
-                <mesh filename="file://$(find robo_arm)/meshes/Link_4.STL" />
-            </geometry>
-            <material name="">
-                <color rgba="0.90 0.35 0.117 1" />
-            </material>
-        </visual>
-        <collision>
-            <origin xyz="0 0 0" rpy="0 0 0" />
-            <geometry>
-                <mesh filename="file://$(find robo_arm)/meshes/Link_4.STL" />
-            </geometry>
-        </collision>
-    </link>
+    <link name="Link_3">
+        <inertial>
+            <origin xyz="1.56358976851345E-05 -0.000283205718507318 -0.0822589976475606" rpy="0 0 0" />
+            <mass value="0.0846391903579548" />
+            <inertia ixx="0.000140247302733448" ixy="-4.69358368842248E-12"
+                ixz="-3.07601656051575E-07" iyy="0.000127934879343709" iyz="-1.64072771614451E-07"
+                izz="3.08569655735298E-05" />
+        </inertial>
+        <visual>
+            <origin xyz="0 0 0" rpy="0 0 0" />
+            <geometry>
+                <mesh filename="file://$(find robo_arm)/meshes/Link_3.STL" />
+            </geometry>
+            <material name="orange" />
+        </visual>
+        <collision>
+            <origin xyz="0 0 0" rpy="0 0 0" />
+            <geometry>
+                <mesh filename="file://$(find robo_arm)/meshes/Link_3.STL" />
+            </geometry>
+        </collision>
+    </link>
+    <gazebo reference="Link_3">
+        <material>Gazebo/Orange</material>
+    </gazebo>
+    <!-- JOINT 4 -->
     <joint name="Joint_4" type="revolute">
         <origin xyz="0 0 -0.12503" rpy="-0.88402 0 1.5708" />
@@ -153,26 +159,30 @@
         <limit lower="-2.3" upper="1" effort="10" velocity="50" />
     </joint>
-    <link name="End_Effector">
-<inertial>
-            <origin xyz="-0.0410338250877696 0.00230286861801432 0.00425320117288218" rpy="0 0 0" />
-            <mass value="0.0486239972257278" />
-            <inertia ixx="8.01424949641006E-06" ixy="2.26577983146827E-07" ixz="4.03073122467701E-07" iyy="1.72794175621324E-05" iyz="2.87107880228718E-07" izz="1.26363118173937E-05" />
-        </inertial>
-        <visual>
-            <origin xyz="0 0 0" rpy="0 0 0" />
-            <geometry>
-                <mesh filename="file://$(find robo_arm)/meshes/End_Effector.STL" />
-            </geometry>
-            <material name="">
-                <color rgba="1 1 1 1" />
-            </material>
-        </visual>
-        <collision>
-            <origin xyz="0 0 0" rpy="0 0 0" />
-            <geometry>
-                <mesh filename="file://$(find robo_arm)/meshes/End_Effector.STL" />
-            </geometry>
-        </collision>
-    </link>
+    <link name="Link_4">
+        <inertial>
+            <origin xyz="-0.000290289833333423 0.0355291858374829 0.00215430200212582" rpy="0 0 0" />
+            <mass value="0.0395556566949035" />
+            <inertia ixx="2.27747448686024E-05" ixy="-1.15013948411467E-07"
+                ixz="-7.6137139609455E-10" iyy="1.92306725633858E-05" iyz="-3.31159527434926E-07"
+                izz="3.22545102910992E-05" />
+        </inertial>
+        <visual>
+            <origin xyz="0 0 0" rpy="0 0 0" />
+            <geometry>
+                <mesh filename="file://$(find robo_arm)/meshes/Link_4.STL" />
+            </geometry>
+            <material name="orange" />
+        </visual>
+        <collision>
+            <origin xyz="0 0 0" rpy="0 0 0" />
+            <geometry>
+                <mesh filename="file://$(find robo_arm)/meshes/Link_4.STL" />
+            </geometry>
+        </collision>
+    </link>
+    <gazebo reference="Link_4">
+        <material>Gazebo/Orange</material>
+    </gazebo>
+    <!-- JOINT 5 -->
     <joint name="Joint_5" type="revolute">
         <origin xyz="-0.0002 0.059362 -0.0026" rpy="-1.6304 0 -1.5708" />
@@ -182,5 +192,30 @@
         <limit lower="-3.14" upper="0" effort="10" velocity="50" />
     </joint>
-<transmission name="trans_Joint_1">
+    <link name="End_Effector">
+        <inertial>
+            <origin xyz="-0.0410338250877696 0.00230286861801432 0.00425320117288218" rpy="0 0 0" />
+            <mass value="0.0486239972257278" />
+            <inertia ixx="8.01424949641006E-06" ixy="2.26577983146827E-07"
+                ixz="4.03073122467701E-07" iyy="1.72794175621324E-05" iyz="2.87107880228718E-07"
+                izz="1.26363118173937E-05" />
+        </inertial>
+        <visual>
+            <origin xyz="0 0 0" rpy="0 0 0" />
+            <geometry>
+                <mesh filename="file://$(find robo_arm)/meshes/End_Effector.STL" />
+            </geometry>
+            <material name="white" />
+        </visual>
+        <collision>
+            <origin xyz="0 0 0" rpy="0 0 0" />
+            <geometry>
+                <mesh filename="file://$(find robo_arm)/meshes/End_Effector.STL" />
+            </geometry>
+        </collision>
+    </link>
+    <gazebo reference="End_Effector">
+        <material>Gazebo/White</material>
+    </gazebo>
+    <transmission name="trans_Joint_1">
         <type>transmission_interface/SimpleTransmission</type>
         <joint name="Joint_1">
@@ -232,4 +267,5 @@
         </actuator>
     </transmission>
+    <!-- ROS CONTROL -->
     <gazebo>
         <plugin name="gazebo_ros_control" filename="libgazebo_ros_control.so">

Commit message: update 20231112

File: urdf/robot_assembly(gazebo).xacro (robot description, xacro)
@@ -9,5 +9,6 @@
     <xacro:property name="height" value="2" />
     <xacro:property name="axle_offset" value="0.05" />
-    <xacro:property name="damp" value="0.7" />
+    <xacro:property name="damping" value="0.5" />
+    <xacro:property name="friciton" value="100" />
     <!-- Materials -->
     <material name="white">
@@ -60,4 +61,5 @@
         <axis xyz="0 0 1" />
         <limit lower="-1.57" upper="1.57" effort="10" velocity="50" />
+        <dynamics damping="${damping}" friction="${friciton}"/>
     </joint>
     <link name="Link_1">
@@ -93,4 +95,5 @@
         <axis xyz="0 1 0" />
         <limit lower="-1.65" upper="0.35" effort="10" velocity="50" />
+        <dynamics damping="${damping}" friction="${friciton}"/>
     </joint>
     <link name="Link_2">
@@ -125,4 +128,5 @@
         <axis xyz="0 1 0" />
         <limit lower="-3.14" upper="0.14" effort="10" velocity="50" />
+        <dynamics damping="${damping}" friction="${friciton}"/>
     </joint>
     <link name="Link_3">
@@ -158,4 +162,5 @@
         <axis xyz="1 0 0" />
         <limit lower="-2.3" upper="1" effort="10" velocity="50" />
+        <dynamics damping="${damping}" friction="${friciton}"/>
     </joint>
     <link name="Link_4">
@@ -191,4 +196,5 @@
         <axis xyz="1 0 0" />
         <limit lower="-3.14" upper="0" effort="10" velocity="50" />
+        <dynamics damping="${damping}" friction="${friciton}"/>
     </joint>
     <link name="End_Effector">
@@ -218,4 +224,5 @@
     </gazebo>
     <!-- Transmission elements -->
+    <!--
     <transmission name="trans_Joint_1">
         <type>transmission_interface/SimpleTransmission</type>
@@ -268,6 +275,7 @@
         </actuator>
     </transmission>
+    -->
     <gazebo>
-        <pluging name="gazebo_ros_joint_state_publisher" filename="libgazebo_ros_joint_state_publisher.so">
+        <plugin name="gazebo_ros_joint_state_publisher" filename="libgazebo_ros_joint_state_publisher.so">
             <update_rate>20</update_rate>
             <joint_name>Joint_1</joint_name>
@@ -276,5 +284,47 @@
             <joint_name>Joint_4</joint_name>
             <joint_name>Joint_5</joint_name>
-        </pluging>
+        </plugin>
+    </gazebo>
+    <!-- ros2 topic pub -1 /set_joint_trajectory trajectory_msgs/msg/JointTrajectory  '{header: {frame_id: world}, joint_names: [Joint_1, Joint_2, Joint_3,_Joint_4, Joint_5], points: [  {positions: {-0.4, 0.7, 0.5, 1.2, 0.5}} ]}' -->
+    <gazebo>
+        <plugin name="gazebo_ros_joint_pose_trajectory"
+            filename="libgazebo_ros_joint_pose_trajectory.so">
+            <update_rate>2</update_rate>
+        </plugin>
+    </gazebo>
+    <joint name="camera_optical_joint" type="fixed">
+        <origin xyz="-0.05 0.05 0" rpy="1.57 0 -3.14159" />
+        <parent link="End_Effector" />
+        <child link="camera_link_optical" />
+        <axis xyz="0 0 0" />
+    </joint>
+    <link name="camera_link_optical"></link>
+    <gazebo reference="camera_link_optical">
+        <sensor type="depth" name="my_cam">
+            <update_rate>20</update_rate>
+            <visualize>true</visualize>
+            <camera name="cam">
+                <horizontal_fov>1.3962634</horizontal_fov>
+                <image>
+                    <width>640</width>
+                    <height>480</height>
+                    <format>R8B8G8</format>
+                </image>
+                <clip>
+                    <near>0.02</near>
+                    <far>300</far>
+                </clip>
+                <noise>
+                    <type>gaussian</type>
+                    <mean>0.0</mean>
+                    <stddev>0.007</stddev>
+                </noise>
+            </camera>
+            <plugin name="camera_controller" filename="libgazebo_ros_camera.so">
+                <frame_name>camera_link_optical</frame_name>
+                <min_depth>0.1</min_depth>
+                <max_depth>500</max_depth>
+            </plugin>
+        </sensor>
     </gazebo>
 </robot>

File: urdf/robot_core.xacro (robot description, xacro)
@@ -2,4 +2,6 @@
 <robot xmlns:xacro="http://www.ros.org/wiki/xacro" name="robot">
     <xacro:include filename="robot_assembly(gazebo).xacro" />
+    <!--
     <xacro:include filename="gazebo_control.xacro" />
+    -->
 </robot>

Commit message: 240201

File: urdf/robot_assembly(gazebo).xacro (robot description, xacro)
@@ -1,7 +1,3 @@
 <?xml version="1.0" encoding="utf-8"?>
-<!-- This URDF was automatically created by SolidWorks to URDF Exporter! Originally created by
-Stephen Brawner (brawner@gmail.com)
-     Commit Version: 1.6.0-4-g7f85cfe  Build Version: 1.6.7995.38578
-     For more information, please see http://wiki.ros.org/sw_urdf_exporter -->
 <robot name="robot_assembly" xmlns:xacro="http://www.ros.org/wiki/xacro">
     <!-- Constants for robot dimensions-->

File: urdf/robot_assembly(moveit) copy.urdf (robot description, URDF)
Before this commit: robot robot_assembly, 7 links, 6 joints
Links:
- link End_Effector: geometry collision mesh filename=package://robo_arm/meshes/End_Effector.STL; visual mesh filename=package://robo_arm/meshes/End_Effector.STL
- link Link_1: geometry collision mesh filename=package://robo_arm/meshes/Link_1.STL; visual mesh filename=package://robo_arm/meshes/Link_1.STL
- link Link_2: geometry collision mesh filename=package://robo_arm/meshes/Link_2.STL; visual mesh filename=package://robo_arm/meshes/Link_2.STL
- link Link_3: geometry collision mesh filename=package://robo_arm/meshes/Link_3.STL; visual mesh filename=package://robo_arm/meshes/Link_3.STL
- link Link_4: geometry collision mesh filename=package://robo_arm/meshes/Link_4.STL; visual mesh filename=package://robo_arm/meshes/Link_4.STL
- link base_link: geometry collision mesh filename=package://robo_arm/meshes/base_link.STL; visual mesh filename=package://robo_arm/meshes/base_link.STL
Joints:
- joint Joint_1: limit lower=-1.57 upper=1.57 effort=10 velocity=50 -> lower=-1.57 upper=1.57 effort=87 velocity=3
- joint Joint_2: limit lower=-1.65 upper=0.35 effort=10 velocity=50 -> lower=-1.65 upper=0.35 effort=87 velocity=3
- joint Joint_3: limit lower=-3.14 upper=0.14 effort=10 velocity=50 -> lower=-3.14 upper=0.14 effort=87 velocity=3
- joint Joint_4: limit lower=-2.3 upper=1 effort=10 velocity=50 -> lower=-2.3 upper=1 effort=87 velocity=3
- joint Joint_5: limit lower=-3.14 upper=0 effort=10 velocity=50 -> lower=-3.14 upper=0.2 effort=87 velocity=3

File: urdf/robot_assembly(moveit).urdf (robot description, URDF)
Before this commit: robot robot_assembly, 7 links, 6 joints
Links:
- link End_Effector: geometry collision mesh filename=package://robo_arm/meshes/End_Effector.STL; visual mesh filename=package://robo_arm/meshes/End_Effector.STL
- link Link_1: geometry collision mesh filename=package://robo_arm/meshes/Link_1.STL; visual mesh filename=package://robo_arm/meshes/Link_1.STL
- link Link_2: geometry collision mesh filename=package://robo_arm/meshes/Link_2.STL; visual mesh filename=package://robo_arm/meshes/Link_2.STL
- link Link_3: geometry collision mesh filename=package://robo_arm/meshes/Link_3.STL; visual mesh filename=package://robo_arm/meshes/Link_3.STL
- link Link_4: geometry collision mesh filename=package://robo_arm/meshes/Link_4.STL; visual mesh filename=package://robo_arm/meshes/Link_4.STL
- link base_link: geometry collision mesh filename=package://robo_arm/meshes/base_link.STL; visual mesh filename=package://robo_arm/meshes/base_link.STL
Joints:
- joint Joint_1: limit lower=-1.57 upper=1.57 effort=10 velocity=50 -> lower=-1.57 upper=1.57 effort=87 velocity=3
- joint Joint_2: limit lower=-1.65 upper=0.35 effort=10 velocity=50 -> lower=-1.65 upper=0.35 effort=87 velocity=3
- joint Joint_3: limit lower=-3.14 upper=0.14 effort=10 velocity=50 -> lower=-3.14 upper=0.14 effort=87 velocity=3
- joint Joint_4: limit lower=-2.3 upper=1 effort=10 velocity=50 -> lower=-2.3 upper=1 effort=87 velocity=3
- joint Joint_5: limit lower=-3.14 upper=0 effort=10 velocity=50 -> lower=-3.14 upper=0.2 effort=87 velocity=3
